Commit message: gazeboでgmappingができない問題の修正

File: configuration_files/cartographer/mecanumrover_cartographer.urdf (robot description, URDF)
Before this commit: robot megarover, 2 links, 1 joints
Links:
- removed link horizontal_laser_link
- added link lidar_link; visual cylinder length=0.05 radius=0.03
Joints:
- removed joint horizontal_laser_link_joint
- added joint lidar_link_joint: type fixed, parent base_link, child lidar_link, origin xyz=0.199 0 0.06 rpy=3.14159 0.0 0.0

File: urdf/vmecanumrover.xacro (robot description, xacro)
@@ -380,18 +380,18 @@
   <!-- back -->
   <xacro:bumperbaseboard prefix="back" parent="body_link" xyz="-0.196 0 0.0365" z_dir="-90"/>
-  <!-- base attachment(LiDER,emergency button,wyreless charge) board(front) -->
+  <!-- base attachment(LiDAR,emergency button,wyreless charge) board(front) -->
   <!--  upper side  -->
 <!--  <xacro:optionattachboard prefix="front" xyz="0.157 0 0.1665" z_dir="0" /> -->
   <!--  lower side  -->
   <xacro:optionattachboard prefix="front" xyz="0.157 0 0.1585" z_dir="0" />
-  <!-- base attachment(LiDER,emergency button,wyreless charge) board(back) -->
+  <!-- base attachment(LiDAR,emergency button,wyreless charge) board(back) -->
   <!--  upper side  -->
 <!--  <xacro:optionattachboard prefix="back" xyz="-0.157 0 0.1665" z_dir="180" /> -->
   <!--  lower side  -->
   <xacro:optionattachboard prefix="back" xyz="-0.157 0 0.1585" z_dir="180" />
-  <!-- LiDER  -->
-  <joint name="lider_joint" type="fixed">
+  <!-- LiDAR  -->
+  <joint name="lidar_joint" type="fixed">
     <parent link="board_front_link"/>
-    <child  link="lider_link"/>
+    <child  link="lidar_link"/>
   <!-- attach upper side -->
 <!--    <origin xyz="0.042 0 0.0570" rpy="0 0 0"/> -->
@@ -399,8 +399,8 @@
     <origin xyz="0.042 0 -0.0570" rpy="${radians(180)} 0 0"/>
   </joint>
-  <link name="lider_link">
-    <visual>
-      <geometry>
-          <mesh filename="package://mecanumrover_samples/meshes/dae/mecanum_lider.dae" />
+  <link name="lidar_link">
+    <visual>
+      <geometry>
+          <mesh filename="package://mecanumrover_samples/meshes/dae/mecanum_lidar.dae" />
       </geometry>
       <material name="black"/>
@@ -408,5 +408,5 @@
     <collision>
       <geometry>
-          <mesh filename="package://mecanumrover_samples/meshes/stl/mecanum_lider.stl" />
+          <mesh filename="package://mecanumrover_samples/meshes/stl/mecanum_lidar.stl" />
       </geometry>
     </collision>
@@ -415,7 +415,7 @@
     </inertial>
   </link>
-  <gazebo reference="lider_link">
+  <gazebo reference="lidar_link">
     <material>Gazebo/Black</material>
-    <sensor type="ray" name="lrf_sensor">
+    <sensor type="ray" name="lidar_sensor">
       <pose>0 0 0 0 0 0</pose>
       <visualize>true</visualize>
@@ -443,5 +443,5 @@
       <plugin name="gazebo_ros_lrf_controller" filename="libgazebo_ros_laser.so">
         <topicName>/scan</topicName>
-        <frameName>laser</frameName>
+        <frameName>lidar_link</frameName>
       </plugin>
     </sensor>
